File: v1.0/PCB/DIP-HDMI-v1.0.sch (EAGLE design)
At the start: 59 parts, among them J1 T_MOLEX_45171, J2 2X20CHIP, J3 HDR2X5, J4 HDR2X3, J5 HDR1X8, J6 HDR2X8, J7 HDR1X2, U1 CH7053A, U2 LP5907MFX, U3 DS2431P+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

Commit message: added datasheets and layer stack up
Other:
- moved on the sheet: C1, C10, C11, C12, C13, C14, C15, C16, C17, C18, C19, C2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
